File: project/PCB-MachineThatDraws/PCB-MachineThatDraws.kicad_pcb (KiCad board)
At the start: 2 copper layers, 29 parts, among them J2 Barrel_Jack_Switch, J3 Switch, J4 Switch, J5 Moteur, J6 Moteur, J7 Arret urgence, J8 Servo-Moteur, U2 R-78E5.0-1.0

Commit message: Faire PCB
Parts:
- removed JP1, JP2, JP3, JP4, JP5, JP6: Microstep Resolution, Jumper:Jumper_Harwin_S1621_P10.9mm
- added J1: SD_Card_Device, Connector_Card:SD_Card_Device_16mm_SlotDepth, F.Cu at (237.8, 86.5)
- added J10: Conn_02x03_Counter_Clockwise, Connector_PinHeader_2.54mm:PinHeader_2x03_P2.54mm_Vertical, F.Cu at (199.2, 55.0)
- added J9: Conn_02x03_Counter_Clockwise, Connector_PinHeader_2.54mm:PinHeader_2x03_P2.54mm_Vertical, F.Cu at (225.8, 60.0)
- added R6: 10K, makerspace-unilasalle:R_1206, F.Cu at (242.0, 107.0)
- added R7: 10K, makerspace-unilasalle:R_1206, F.Cu at (248.0, 103.5)
- added U1: ESP32-S3-UNO, makerspace-unilasalle:ESP_S3_UNO, F.Cu at (206.8, 99.6)
- C3, C4: footprint Capacitor_SMD:CP_Elec_3x5.3 -> Capacitor_SMD:CP_Elec_6.3x5.4
- D1: footprint LED_THT:LED_D3.0mm_FlatTop -> LED_SMD:LED_1206_3216Metric
- Display1, J5, J6: footprint Connector_JST:JST_EH_B4B-EH-A_1x04_P2.50mm_Vertical -> Connector_PinHeader_2.54mm:PinHeader_1x04_P2.54mm_Vertical
- F1: footprint Fuse:Fuse_0402_1005Metric -> Fuse:Fuseholder_Blade_Mini_Keystone_3568
- J2: footprint Connector_BarrelJack:BarrelJack_CUI_PJ-036AH-SMT_Horizontal -> Connector_BarrelJack:BarrelJack_GCT_DCJ200-10-A_Horizontal
- J3, J4, J8: footprint Connector_JST:JST_PH_B3B-PH-K_1x03_P2.00mm_Vertical -> Connector_PinHeader_2.54mm:PinHeader_1x03_P2.54mm_Vertical
- J7: footprint TerminalBlock_Ningbo-Kagnex:TerminalBlock_Ningbo-Kagnex_HB9500M_1x02_P9.5mm -> TerminalBlock:TerminalBlock_bornier-2_P5.08mm
- R3, R4, R5: footprint makerspace-unilasalle:R_Axial -> makerspace-unilasalle:R_1206
- moved R5 153.0 mm to (198.5, 79.0)
- moved R4 152.1 mm to (198.5, 76.5)
- moved J3 148.2 mm to (243.0, 103.5), turned to -90 degrees
- moved C2 147.3 mm to (200.3, 83.0)
- moved C8 147.3 mm to (197.0, 83.0)
- moved Display1 138.7 mm to (203.7, 76.5), turned to 0 degrees
- moved A1 113.1 mm to (218.3, 72.4)
- moved C7 112.4 mm to (200.5, 94.5), turned to 90 degrees
- moved J4 110.4 mm to (228.5, 103.5), turned to 90 degrees
- moved J8 109.2 mm to (204.0, 98.5), turned to 180 degrees
- moved J5 105.7 mm to (222.0, 71.5), turned to 180 degrees
- moved J2 102.1 mm to (211.3, 76.7)
- moved A2 96.8 mm to (241.8, 72.2)
- moved C4 96.3 mm to (251.0, 55.5), turned to -90 degrees
- moved J6 92.8 mm to (245.4, 67.2), turned to 180 degrees
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Routing:
- net Net-(J7-Pin_2): track 0.00 -> 0.54 mm
Other:
- board outline added: 16 x 24 mm

Commit message: A refaire
Parts:
- moved C5 41.0 mm to (253.1, 104.3)
- moved J8 32.4 mm to (235.5, 106.0), turned to -90 degrees
- moved C7 25.0 mm to (225.5, 93.9), turned to 0 degrees
- moved J2 19.1 mm to (230.3, 78.1)
- moved U2 18.6 mm to (219.5, 106.3)
- moved F1 18.4 mm to (209.5, 89.5)
- moved R7 17.5 mm to (232.0, 96.5), turned to 0 degrees
- moved R6 16.3 mm to (232.0, 94.1)
- moved J4 13.0 mm to (241.0, 107.0), turned to 180 degrees
- moved D1 11.6 mm to (215.0, 96.0), turned to 0 degrees
- moved C6 11.2 mm to (225.5, 96.5), turned to 0 degrees
- moved J3 3.86 mm to (244.7, 107.0), turned to 180 degrees
- moved R3 3.00 mm to (220.5, 96.0), turned to 0 degrees
- moved J7 1.04 mm to (221.0, 84.4)
- moved J1 0.35 mm to (237.8, 86.1)
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Routing:
- net GND: track 0.00 -> 207.3 mm, vias 0 -> 5
- net +3.3V: track 0.02 -> 60.5 mm, vias 0 -> 3
- net D19: track 0.00 -> 38.2 mm, vias 0 -> 1
- net +5V: track 0.00 -> 22.7 mm, vias 0 -> 1
- net D17: track 0.00 -> 21.1 mm
- net D05: track 0.00 -> 18.6 mm, vias 0 -> 1
- net D02: track 0.00 -> 13.7 mm
- net +12V: track 0.42 -> 13.3 mm, vias 0 -> 1
- net Net-(J7-Pin_1): track 0.00 -> 12.0 mm
- net Net-(J7-Pin_2): track 0.54 -> 11.5 mm
- net Net-(A1-MS2): track 0.00 -> 7.03 mm
- net Net-(A2-MS3): track 0.00 -> 4.13 mm
- net SCL : track 0.00 -> 4.04 mm, vias 0 -> 1
- net SDA: track 0.06 -> 4.05 mm, vias 0 -> 1
- net Net-(A2-MS1): track 0.00 -> 3.65 mm
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
Commit message: A repenser
Parts:
- moved C5 112.9 mm to (141.4, 120.2), turned to 180 degrees
- moved J3 84.1 mm to (161.8, 120.8)
- moved J4 83.8 mm to (158.0, 118.1)
- moved C7 73.5 mm to (153.3, 107.4)
- moved R6 73.5 mm to (159.8, 107.6)
- moved A1 73.5 mm to (146.1, 85.9)
- moved A2 73.5 mm to (169.6, 85.5)
- moved C2 73.5 mm to (128.1, 96.5)
- moved C3 73.5 mm to (127.3, 81.5)
- moved C4 73.5 mm to (178.8, 69.0)
- moved C6 73.5 mm to (153.3, 110.0)
- moved C8 73.5 mm to (124.8, 96.5)
- moved D1 73.5 mm to (142.8, 109.5)
- moved Display1 73.5 mm to (131.8, 90.0)
- moved F1 73.5 mm to (137.3, 103.0)
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Routing:
- net GND: track 207.3 -> 0.24 mm, vias 5 -> 0
- net +3.3V: track 60.5 -> 0.00 mm, vias 3 -> 0
- net D19: track 38.2 -> 0.00 mm, vias 1 -> 0
- net +5V: track 22.7 -> 0.00 mm, vias 1 -> 0
- net D17: track 21.1 -> 0.00 mm
- net D05: track 18.6 -> 0.00 mm, vias 1 -> 0
- net D02: track 13.7 -> 0.00 mm
- net +12V: track 13.3 -> 0.00 mm, vias 1 -> 0
- net Net-(J7-Pin_1): track 12.0 -> 0.00 mm
- net Net-(J7-Pin_2): track 11.5 -> 0.00 mm
- net Net-(A1-MS2): track 7.03 -> 0.01 mm
- net Net-(A2-MS3): track 4.13 -> 0.00 mm
- net SDA: track 4.05 -> 0.00 mm, vias 1 -> 0
- net SCL : track 4.04 -> 0.00 mm, vias 1 -> 0
- net Net-(A2-MS1): track 3.65 -> 0.00 mm
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Other:
- board size 16 x 24 mm -> 60 x 60 mm

Commit message: Finale
Routing:
- net +12V: track 0.00 -> 70.8 mm
- net +3.3V: track 0.00 -> 58.7 mm, vias 0 -> 2
- net D11: track 0.00 -> 56.3 mm
- net D18: track 0.00 -> 39.9 mm, vias 0 -> 2
- net D19: track 0.00 -> 36.7 mm, vias 0 -> 2
- net +5V: track 0.00 -> 32.2 mm
- net D12: track 0.00 -> 24.9 mm
- net D03: track 0.00 -> 22.9 mm, vias 0 -> 1
- net D17: track 0.00 -> 22.7 mm, vias 0 -> 1
- net D05: track 0.00 -> 21.8 mm
- net D13: track 0.00 -> 21.8 mm
- net Net-(J7-Pin_2): track 0.00 -> 12.1 mm
- net Net-(J7-Pin_1): track 0.00 -> 11.8 mm
- net Net-(A1-MS3): track 0.00 -> 10.6 mm
- net Net-(A1-MS1): track 0.00 -> 7.32 mm
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- added copper zone on F.Cu, net +12V
- added copper zone on B.Cu, net +3.3V
- added copper zone on F.Cu, net +3.3V
- added copper zone on F.Cu, net +5V
- added copper zone on B.Cu, net GND
- added copper zone on F.Cu, net GND

Commit message: petites modifications apportées
Routing:
- net +3.3V: track 58.7 -> 116.6 mm
- net +12V: track 70.8 -> 100.3 mm
Changed lines of the file:
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@@
 	)
 	(segment
-		(start 136.785375 92.5855)
-		(end 135.087904 90.888029)
+		(start 143 78.75)
+		(end 143 71.23)
+		(width 0.73057)
+		(layer "F.Cu")
+		(net 5)
+	)
+	(segment
+		(start 129.284846 87.254971)
+		(end 127.798502 85.768627)
+		(width 0.73057)
+		(layer "F.Cu")
+		(net 5)
+	)
+	(segment
+		(start 137.279875 94.820714)
+		(end 137.279875 93.08)
+		(width 0.73057)
+		(layer "F.Cu")
+		(net 5)
+	)
+	(segment
+		(start 135.253084 113.391473)
+		(end 135.253084 96.847506)
 		(width 0.73057)
 		(layer "F.Cu")
@@
 	)
 	(segment
-		(start 135.087904 90.888029)
-		(end 135.087904 90.661174)
+		(start 131.754971 87.254971)
+		(end 129.284846 87.254971)
+		(width 0.73057)
+		(layer "F.Cu")
+		(net 5)
+	)
+	(segment
+		(start 133.5 88.25)
+		(end 143 78.75)
 		(width 0.73057)
 		(layer "F.Cu")
@@
 	)
 	(segment
+		(start 143 71.23)
+		(end 146.12 68.11)
+		(width 0.73057)
+		(layer "F.Cu")
+		(net 5)
+	)
+	(segment
 		(start 137.279875 93.08)
-		(end 137.279875 94.820714)
+		(end 136.785375 92.5855)
+		(width 0.73057)
+		(layer "F.Cu")
+		(net 5)
+	)
+	(segment
+		(start 133.5 89)
+		(end 133.5 88.25)
 		(width 0.73057)
 		(layer "F.Cu")
@@
 	)
 	(segment
-		(start 141.061904 118.076029)
-		(end 142.468699 119.482824)
-		(width 0.73057)
-		(layer "F.Cu")
-		(net 5)
-	)
-	(segment
-		(start 137.279875 94.820714)
-		(end 135.253084 96.847506)
-		(width 0.73057)
-		(layer "F.Cu")
-		(net 5)
-	)
-	(segment
-		(start 131.681701 87.254971)
-		(end 129.284846 87.254971)
-		(width 0.73057)
-		(layer "F.Cu")
-		(net 5)
-	)
-	(segment
 		(start 149.371411 66.25)
 		(end 147.980375 66.25)
@@
 	)
 	(segment
-		(start 135.087904 90.661174)
-		(end 131.681701 87.254971)
+		(start 142.841375 120.1805)
+		(end 142.468699 119.482824)
 		(width 0.73057)
 		(layer "F.Cu")
@@
 	)
 	(segment
-		(start 135.253084 96.847506)
-		(end 135.253084 113.391473)
-		(width 0.73057)
-		(layer "F.Cu")
-		(net 5)
-	)
-	(segment
-		(start 129.284846 87.254971)
-		(end 127.798502 85.768627)
+		(start 136.785375 92.285375)
+		(end 133.5 89)
 		(width 0.73057)
 		(layer "F.Cu")
@@
 	(segment
 		(start 139.93764 118.076029)
+		(end 135.253084 113.391473)
+		(width 0.73057)
+		(layer "F.Cu")
+		(net 5)
+	)
+	(segment
+		(start 135.253084 96.847506)
+		(end 137.279875 94.820714)
+		(width 0.73057)
+		(layer "F.Cu")
+		(net 5)
+	)
+	(segment
+		(start 136.785375 92.5855)
+		(end 136.785375 92.285375)
+		(width 0.73057)
+		(layer "F.Cu")
+		(net 5)
+	)
+	(segment
+		(start 140.68 93.08)
+		(end 137.28 93.08)
+		(width 0.73057)
+		(layer "F.Cu")
+		(net 5)
+	)
+	(segment
+		(start 141.061904 118.076029)
+		(end 139.93764 118.076029)
+		(width 0.73057)
+		(layer "F.Cu")
+		(net 5)
+	)
+	(segment
+		(start 142.468699 119.482824)
 		(end 141.061904 118.076029)
 		(width 0.73057)
@@
 	)
 	(segment
-		(start 137.279875 93.08)
-		(end 136.785375 92.5855)
-		(width 0.73057)
-		(layer "F.Cu")
-		(net 5)
-	)
-	(segment
-		(start 142.468699 119.482824)
-		(end 142.841375 120.1805)
-		(width 0.73057)
-		(layer "F.Cu")
-		(net 5)
-	)
-	(segment
-		(start 135.253084 113.391473)
-		(end 139.93764 118.076029)
+		(start 133.5 89)
+		(end 131.754971 87.254971)
 		(width 0.73057)
 		(layer "F.Cu")
@@
 	)
 	(segment
+		(start 124.78 95.025)
+		(end 128.13 95.025)
+		(width 0.254)
+		(layer "F.Cu")
+		(net 7)
+	)
+	(segment
+		(start 129.545 73.555)
+		(end 127.005 73.555)
+		(width 0.254)
+		(layer "F.Cu")
+		(net 7)
+	)
+	(segment
 		(start 159.400863 106.186012)
 		(end 165.714002 99.872873)
@@
 	)
 	(segment
+		(start 127.005 73.555)
+		(end 124.8175 75.7425)
+		(width 0.254)
+		(layer "F.Cu")
+		(net 7)
+	)
+	(segment
+		(start 169.12 83.5)
+		(end 167 83.5)
+		(width 0.254)
+		(layer "F.Cu")
+		(net 7)
+	)
+	(segment
 		(start 165.714002 99.872873)
 		(end 172.040753 99.872873)
@@
 	)
 	(segment
+		(start 128.13 95.025)
+		(end 128.525 95.025)
+		(width 0.254)
+		(layer "F.Cu")
+		(net 7)
+	)
+	(segment
 		(start 169.335485 82.71511)
 		(end 168.521887 81.901512)
@@
 	)
 	(segment
+		(start 169.62 83)
+		(end 169.12 83.5)
+		(width 0.254)
+		(layer "F.Cu")
+		(net 7)
+	)
+	(segment
 		(start 168.521887 81.901512)
 		(end 158.190375 71.57)
@@
 	)
 	(segment
+		(start 164.5 92)
+		(end 172.040753 99.540753)
+		(width 0.254)
+		(layer "F.Cu")
+		(net 7)
+	)
+	(segment
 		(start 154.931443 70.032966)
 		(end 154.931443 69.820631)
@@
 	)
 	(segment
+		(start 172.040753 99.540753)
+		(end 172.040753 99.872873)
+		(width 0.254)
+		(layer "F.Cu")
+		(net 7)
+	)
+	(segment
 		(start 150.712375 71.2875)
 		(end 149.880887 72.118988)
@@
 	)
 	(segment
+		(start 124.78 90.0375)
+		(end 124.8175 90)
+		(width 0.254)
+		(layer "F.Cu")
+		(net 7)
+	)
+	(segment
 		(start 154.931443 69.820631)
 		(end 154.689582 69.57877)
@@
 	)
 	(segment
+		(start 167 83.5)
+		(end 164.5 86)
+		(width 0.254)
+		(layer "F.Cu")
+		(net 7)
+	)
+	(segment
 		(start 148.424285 73.57559)
 		(end 148.424285 81.04609)
@@
 	)
 	(segment
+		(start 128.54 95.04)
+		(end 131.78 95.04)
+		(width 0.254)
+		(layer "F.Cu")
+		(net 7)
+	)
+	(segment
+		(start 128.525 95.025)
+		(end 128.54 95.04)
+		(width 0.254)
+		(layer "F.Cu")
+		(net 7)
+	)
+	(segment
+		(start 124.78 95.025)
+		(end 124.78 90.0375)
+		(width 0.254)
+		(layer "F.Cu")
+		(net 7)
+	)
+	(segment
+		(start 124.8175 75.7425)
+		(end 124.8175 90)
+		(width 0.254)
+		(layer "F.Cu")
+		(net 7)
+	)
+	(segment
+		(start 129.545 71.015)
+		(end 129.545 73.555)
+		(width 0.254)
+		(layer "F.Cu")
+		(net 7)
+	)
+	(segment
 		(start 151.014875 70.985)
 		(end 150.712375 71.2875)
@@
 		(layer "F.Cu")
 		(net 7)
+	)
+	(segment
+		(start 164.5 86)
+		(end 164.5 92)
+		(width 0.254)
+		(layer "F.Cu")
+		(net 7)

Commit message: a refaire
Parts:
- moved U2 63.0 mm to (108.2, 71.4), turned to 90 degrees
- moved C6 60.0 mm to (112.0, 66.5), turned to -90 degrees
- moved C5 56.9 mm to (112.0, 71.5), turned to 90 degrees
- moved J2 54.5 mm to (105.5, 105.7)
- moved J7 43.4 mm to (105.5, 101.0), turned to 90 degrees
- moved F1 36.1 mm to (103.8, 89.5)
Routing:
- net +12V: track 100.3 -> 88.2 mm
- net Net-(J7-Pin_2): track 12.1 -> 19.7 mm
- net Net-(J7-Pin_1): track 11.8 -> 4.65 mm
- net +5V: track 32.2 -> 25.1 mm
- net GND: track 0.24 -> 5.88 mm
- net +3.3V: track 116.6 -> 117.0 mm, vias 2 -> 3
- net SDA: track 4.05 -> 4.39 mm, vias 0 -> 1
- net SCL : vias 0 -> 1

Commit message: Peut etre a revoir
Parts:
- J1: footprint Connector_Card:SD_Card_Device_16mm_SlotDepth -> Connector_Card:microSD_HC_Molex_47219-2001
- moved J10 67.2 mm to (178.2, 111.9)
- moved J3 53.4 mm to (191.0, 76.1), turned to -90 degrees
- moved J4 48.7 mm to (191.0, 82.3), turned to -90 degrees
- moved Display1 44.7 mm to (157.5, 126.6), turned to -90 degrees
- moved R4 44.0 mm to (157.5, 121.0), turned to -90 degrees
- moved R5 40.4 mm to (155.0, 121.0), turned to -90 degrees
- moved C3 39.3 mm to (153.2, 111.1)
- moved C7 38.6 mm to (186.9, 88.4), turned to 90 degrees
- moved D1 38.1 mm to (157.8, 74.5), turned to 180 degrees
- moved U2 37.8 mm to (144.8, 80.9)
- moved C5 37.8 mm to (148.6, 81.0)
- moved C6 37.8 mm to (148.6, 76.0)
- moved J7 37.8 mm to (142.1, 110.5)
- moved F1 37.8 mm to (140.4, 98.9)
- moved J2 37.8 mm to (142.1, 115.1)
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Routing:
- net +5V: track 25.1 -> 93.0 mm
- net GND: track 5.88 -> 55.1 mm, vias 60 -> 66
- net D01: track 3.16 -> 46.6 mm, vias 0 -> 2
- net D02: track 2.41 -> 39.6 mm, vias 0 -> 2
- net D07: track 2.71 -> 29.3 mm, vias 0 -> 1
- net +3.3V: track 117.0 -> 142.5 mm, vias 3 -> 0
- net D03: track 22.9 -> 6.01 mm, vias 1 -> 0
- net D05: track 21.8 -> 35.5 mm
- net D11: track 56.3 -> 42.8 mm, vias 0 -> 1
- net D13: track 21.8 -> 31.7 mm
- net D19: track 36.7 -> 27.8 mm, vias 2 -> 0
- net D17: track 22.7 -> 14.7 mm, vias 1 -> 0
- net D12: track 24.9 -> 30.8 mm, vias 0 -> 1
- net +12V: track 88.2 -> 82.4 mm
- net D18: track 39.9 -> 36.0 mm, vias 2 -> 1
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- removed copper zone on F.Cu, net +12V
- removed copper zone on B.Cu, net +3.3V
- removed copper zone on F.Cu, net +3.3V
- removed copper zone on F.Cu, net +5V
