File: project/PCB-MachineThatDraws/PCB-MachineThatDraws.kicad_pcb (KiCad board)
At the start: 2 copper layers, 60 x 60 mm, 29 parts, among them J1 SD_Card_Device, J10 Conn_02x03_Counter_Clockwise, J2 Barrel_Jack_Switch, J3 Switch, J4 Switch, J5 Moteur, J6 Moteur, J7 Arret urgence, J8 Servo-Moteur, J9 Conn_02x03_Counter_Clockwise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

Commit message: Update PCB-MachineThatDraws.kicad_pcb
Routing:
- net D05: track 35.5 -> 40.1 mm
Changed lines of the file:
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@@
 			(at 4.96 -2.67 90)
 			(layer "F.SilkS")
+			(hide yes)
 			(effects
 				(font
@@
 			(layer "F.Fab")
 		)
-		(fp_text user "${REFERENCE}"
-			(at 0 0 90)
-			(layer "F.Fab")
-			(effects
-				(font
-					(size 0.8 0.8)
-					(thickness 0.12)
-				)
-			)
-		)
 		(pad "1" smd roundrect
 			(at -1.4625 0 270)
@@
 		(tags "terminal block bornier2")
 		(property "Reference" "J7"
-			(at 2.54 -5.08 90)
+			(at 2.527625 0.007441 90)
 			(layer "F.SilkS")
 			(effects
@@
 			(layer "F.Fab")
 		)
-		(fp_text user "${REFERENCE}"
-			(at 2.54 0 90)
-			(layer "F.Fab")
-			(effects
-				(font
-					(size 1 1)
-					(thickness 0.15)
-				)
-			)
-		)
 		(pad "1" thru_hole rect
 			(at 0 0 90)
@@
 			(at 0.004801 0.02096 90)
 			(layer "F.SilkS")
+			(hide yes)
 			(effects
 				(font
@@
 		(tags "capacitor")
 		(property "Reference" "C7"
-			(at 0 -1.85 90)
+			(at 0 0 90)
 			(layer "F.SilkS")
+			(hide yes)
 			(effects
 				(font
@@
 		)
 		(fp_text user "${REFERENCE}"
-			(at 0 0 90)
+			(at -0.293006 1.200706 90)
 			(layer "F.Fab")
 			(effects
@@
 			(at 0 0.42 90)
 			(layer "F.SilkS")
+			(hide yes)
 			(effects
 				(font
@@
 			(at -0.0309 -0.063502 0)
 			(layer "F.SilkS")
+			(hide yes)
 			(effects
 				(font
@@
 			(at -0.00633 -0.004294 0)
 			(layer "F.SilkS")
+			(hide yes)
 			(effects
 				(font
@@
 		(tags "Through hole pin header THT 1x03 2.54mm single row")
 		(property "Reference" "J8"
-			(at 38.117135 -37.120009 180)
+			(at -1.200149 3.642145 270)
 			(layer "F.SilkS")
 			(effects
@@
 		(tags "Through hole pin header THT 2x03 2.54mm double row")
 		(property "Reference" "J10"
-			(at 1.27 -2.33 0)
+			(at 1.27 2.531889 90)
 			(layer "F.SilkS")
 			(effects
@@
 			(at -0.003135 0.001 90)
 			(layer "F.SilkS")
+			(hide yes)
 			(effects
 				(font
@@
 			(at 0 -1.85 0)
 			(layer "F.SilkS")
+			(hide yes)
 			(effects
 				(font
@@
 	)
 	(via
-		(at 194.588905 107.747547)
+		(at 194 107.5)
 		(size 0.61021)
 		(drill 0.305105)
@@
 	)
 	(via
-		(at 194.588905 101.687547)
+		(at 194 102)
 		(size 0.61021)
 		(drill 0.305105)
@@
 	)
 	(segment
-		(start 182.53772 116.573977)
-		(end 182.7 116.736257)
+		(start 182.5 119.8)
+		(end 182.7 120)
 		(width 0.254254)
 		(layer "F.Cu")
@@
 	)
 	(segment
-		(start 182.7 116.736257)
-		(end 182.7 120)
+		(start 182.53772 116.573977)
+		(end 182.5 116.611697)
+		(width 0.254254)
+		(layer "F.Cu")
+		(net 27)
+	)
+	(segment
+		(start 182.5 116.611697)
+		(end 182.5 119.8)
 		(width 0.254254)
 		(layer "F.Cu")
@@
 	)
 	(segment
-		(start 178.116774 98.76987)
-		(end 178.141644 98.745)
+		(start 192.86 120)
+		(end 192.86 115.64)
 		(width 1)
 		(layer "F.Cu")
@@
 	)
 	(segment
-		(start 190.05 98.8)
-		(end 190.998103 98.8)
-		(width 0.254254)
-		(layer "F.Cu")
-		(net 40)
-	)
-	(segment
-		(start 178.141644 98.745)
-		(end 189.5 98.745)
+		(start 195.5 99)
+		(end 195.245 98.745)
 		(width 1)
 		(layer "F.Cu")
@@
 	)
 	(segment
-		(start 193.592992 101.39489)
-		(end 193.592992 118.391138)
-		(width 0.254254)
+		(start 195.5 113)
+		(end 195.5 99)
+		(width 1)
 		(layer "F.Cu")
 		(net 40)
 	)
 	(segment
-		(start 193.592992 119.267008)
-		(end 192.86 120)
-		(width 0.254254)
+		(start 192.86 115.64)
+		(end 195.5 113)
+		(width 1)
 		(layer "F.Cu")
 		(net 40)
 	)
 	(segment
-		(start 190.998103 98.8)
-		(end 193.592992 101.39489)
-		(width 0.254254)
+		(start 178.141644 98.745)
+		(end 178.116774 98.76987)
+		(width 1)
 		(layer "F.Cu")
 		(net 40)
 	)
 	(segment
-		(start 193.592992 118.391138)
-		(end 193.592992 119.267008)
-		(width 0.254254)
+		(start 195.245 98.745)
+		(end 178.141644 98.745)
+		(width 1)
 		(layer "F.Cu")
 		(net 40)

Commit message: A verifier
Parts:
- J1: footprint Connector_Card:microSD_HC_Molex_47219-2001 -> makerspace-unilasalle:SD_Hirose_DM1AA_SF_PEJ82; moved to B.Cu
- moved J1 13.3 mm to (199.2, 108.0)
- moved J8 1.03 mm to (191.0, 91.0)
- moved R6 0.39 mm to (178.5, 105.1)
- moved R7 0.39 mm to (178.5, 100.2)
Routing:
- net +5V: track 93.0 -> 163.0 mm
- net D02: track 39.6 -> 68.6 mm, vias 2 -> 0
- net GND: track 55.1 -> 41.9 mm, vias 66 -> 0
- net D12: track 30.8 -> 41.8 mm
- net D11: track 42.8 -> 52.6 mm, vias 1 -> 2
- net D19: track 27.8 -> 35.8 mm, vias 0 -> 2
- net +3.3V: track 142.5 -> 148.5 mm, vias 0 -> 3
- net +12V: track 82.4 -> 88.5 mm
- net D18: track 36.0 -> 41.2 mm, vias 1 -> 2
- net D05: track 40.1 -> 35.3 mm, vias 0 -> 1
- net D01: track 46.6 -> 50.8 mm, vias 2 -> 1
- net Net-(A1-MS3): track 7.05 -> 9.80 mm
- net Net-(A2-MS2): track 7.29 -> 9.26 mm
- net Net-(A2-MS3): track 4.13 -> 5.62 mm
- net Net-(A1-MS1): track 4.66 -> 5.49 mm
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Other:
- board size 60 x 60 mm -> 84.5 x 60 mm

Commit message: fix some wiring problems
Connections:
- U1 pad 8: +5V -> +12V
Routing:
- net +12V: track 88.5 -> 106.5 mm
- net +5V: track 163.0 -> 166.9 mm
